File: PCB/RelayCTRL.sch (EAGLE design)
At the start: 20 parts, among them Q2 BC848 30V 100mA, Q3 IRLML6402, U1 SN74HC4066D

Commit message: fixed pcb error
Connections:
- removed net N$1: B1.*6, R2.2
- net 5V: now also R2.2
- net IR: now also B1.*6
Other:
- moved on the sheet: R2
Changed lines of the file:
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@@
 <attribute name="TP_SIGNAL_NAME" x="95.25" y="-39.37" size="1.778" layer="97" rot="R180"/>
 </instance>
-<instance part="R2" gate="G$1" x="30.48" y="20.32" smashed="yes">
-<attribute name="NAME" x="26.67" y="21.8186" size="1.778" layer="95"/>
-<attribute name="VALUE" x="26.67" y="17.018" size="1.778" layer="96"/>
+<instance part="R2" gate="G$1" x="22.86" y="25.4" smashed="yes" rot="R90">
+<attribute name="NAME" x="21.3614" y="21.59" size="1.778" layer="95" rot="R90"/>
+<attribute name="VALUE" x="26.162" y="21.59" size="1.778" layer="96" rot="R90"/>
 </instance>
 <instance part="R6" gate="G$1" x="22.86" y="15.24" smashed="yes" rot="R90">
@@
 <wire x1="88.9" y1="-38.1" x2="88.9" y2="-33.02" width="0.1524" layer="91"/>
 <label x="88.9" y="-33.02" size="1.778" layer="95" rot="R90" xref="yes"/>
+</segment>
+<segment>
+<pinref part="R2" gate="G$1" pin="2"/>
+<wire x1="22.86" y1="30.48" x2="22.86" y2="33.02" width="0.1524" layer="91"/>
+<label x="22.86" y="33.02" size="1.778" layer="95"/>
 </segment>
 </net>
@@
 </segment>
 </net>
-<net name="N$1" class="0">
-<segment>
-<pinref part="B1" gate="G$1" pin="*6"/>
-<pinref part="R2" gate="G$1" pin="2"/>
-<wire x1="55.88" y1="20.32" x2="35.56" y2="20.32" width="0.1524" layer="91"/>
-</segment>
-</net>
 <net name="3V" class="0">
 <segment>
@@
 <segment>
 <pinref part="R2" gate="G$1" pin="1"/>
-<wire x1="25.4" y1="20.32" x2="22.86" y2="20.32" width="0.1524" layer="91"/>
 <label x="17.78" y="20.32" size="1.778" layer="95" rot="R180" xref="yes"/>
 <pinref part="R6" gate="G$1" pin="2"/>
 <wire x1="22.86" y1="20.32" x2="17.78" y2="20.32" width="0.1524" layer="91"/>
 <junction x="22.86" y="20.32"/>
-</segment>
-<segment>
+<pinref part="B1" gate="G$1" pin="*6"/>
+<wire x1="22.86" y1="20.32" x2="55.88" y2="20.32" width="0.1524" layer="91"/>
+</segment>
+<segment>

Commit message: PCB Update
Parts:
- added Q1: BC848 30V 100mA, SparkFun-DiscreteSemi:TRANS_NPN-MMBT2222AL
- added R7: 1k, rcl:R-EU_R0603
- renumbered 5V to BZ+, BZ to BZ-, G to IR-
Connections:
- new net BZ-: BZ-.TP, Q1.C
- new net N$1: B1.*6, R2.2
- new net N$5: Q1.B, R7.2
- net 5V: no longer R2.2
- net GND: now also Q1.E, U1.3A, U1.4A
- net IR: no longer B1.*6
- net S1: now also R7.1; no longer BZ-.TP
Other:
- moved on the sheet: R2
Changed lines of the file:
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@@
 <part name="B1" library="SparkFun-Boards" deviceset="SPARKFUN_PRO_MICRO" device=""/>
 <part name="OLED128X32" library="pinhead" library_urn="urn:adsk.eagle:library:325" deviceset="PINHD-1X4" device="" package3d_urn="urn:adsk.eagle:package:22407/2"/>
-<part name="BZ" library="testpad" library_urn="urn:adsk.eagle:library:385" deviceset="TP" device="TP15R" package3d_urn="urn:adsk.eagle:package:27968/1"/>
-<part name="5V" library="testpad" library_urn="urn:adsk.eagle:library:385" deviceset="TP" device="TP15R" package3d_urn="urn:adsk.eagle:package:27968/1"/>
-<part name="G" library="testpad" library_urn="urn:adsk.eagle:library:385" deviceset="TP" device="TP15R" package3d_urn="urn:adsk.eagle:package:27968/1"/>
+<part name="BZ-" library="testpad" library_urn="urn:adsk.eagle:library:385" deviceset="TP" device="TP15R" package3d_urn="urn:adsk.eagle:package:27968/1"/>
+<part name="BZ+" library="testpad" library_urn="urn:adsk.eagle:library:385" deviceset="TP" device="TP15R" package3d_urn="urn:adsk.eagle:package:27968/1"/>
+<part name="IR-" library="testpad" library_urn="urn:adsk.eagle:library:385" deviceset="TP" device="TP15R" package3d_urn="urn:adsk.eagle:package:27968/1"/>
 <part name="R2" library="rcl" library_urn="urn:adsk.eagle:library:334" deviceset="R-EU_" device="R0603" package3d_urn="urn:adsk.eagle:package:23555/3" value="10k"/>
 <part name="R6" library="rcl" library_urn="urn:adsk.eagle:library:334" deviceset="R-EU_" device="R0603" package3d_urn="urn:adsk.eagle:package:23555/3" value="10k"/>
+<part name="R7" library="rcl" library_urn="urn:adsk.eagle:library:334" deviceset="R-EU_" device="R0603" package3d_urn="urn:adsk.eagle:package:23555/3" value="1k"/>
+<part name="Q1" library="SparkFun-DiscreteSemi" library_urn="urn:adsk.eagle:library:514" deviceset="TRANS_NPN" device="-MMBT2222AL" package3d_urn="urn:adsk.eagle:package:38446/1" value="BC848 30V 100mA"/>
 </parts>
 <sheets>
@@
 <attribute name="VALUE" x="64.77" y="78.74" size="1.778" layer="96" rot="R180"/>
 </instance>
-<instance part="BZ" gate="G$1" x="78.74" y="-40.64" smashed="yes" rot="R180">
+<instance part="BZ-" gate="G$1" x="78.74" y="-40.64" smashed="yes" rot="R180">
 <attribute name="NAME" x="80.01" y="-41.91" size="1.778" layer="95" rot="R180"/>
 <attribute name="TP_SIGNAL_NAME" x="77.47" y="-39.37" size="1.778" layer="97" rot="R180"/>
 </instance>
-<instance part="5V" gate="G$1" x="88.9" y="-40.64" smashed="yes" rot="R180">
+<instance part="BZ+" gate="G$1" x="88.9" y="-40.64" smashed="yes" rot="R180">
 <attribute name="NAME" x="90.17" y="-41.91" size="1.778" layer="95" rot="R180"/>
 <attribute name="TP_SIGNAL_NAME" x="87.63" y="-39.37" size="1.778" layer="97" rot="R180"/>
 </instance>
-<instance part="G" gate="G$1" x="96.52" y="-40.64" smashed="yes" rot="R180">
+<instance part="IR-" gate="G$1" x="96.52" y="-40.64" smashed="yes" rot="R180">
 <attribute name="NAME" x="97.79" y="-41.91" size="1.778" layer="95" rot="R180"/>
 <attribute name="TP_SIGNAL_NAME" x="95.25" y="-39.37" size="1.778" layer="97" rot="R180"/>
 </instance>
-<instance part="R2" gate="G$1" x="22.86" y="25.4" smashed="yes" rot="R90">
-<attribute name="NAME" x="21.3614" y="21.59" size="1.778" layer="95" rot="R90"/>
-<attribute name="VALUE" x="26.162" y="21.59" size="1.778" layer="96" rot="R90"/>
+<instance part="R2" gate="G$1" x="30.48" y="20.32" smashed="yes">
+<attribute name="NAME" x="26.67" y="21.8186" size="1.778" layer="95"/>
+<attribute name="VALUE" x="26.67" y="17.018" size="1.778" layer="96"/>
 </instance>
 <instance part="R6" gate="G$1" x="22.86" y="15.24" smashed="yes" rot="R90">
 <attribute name="NAME" x="21.3614" y="11.43" size="1.778" layer="95" rot="R90"/>
 <attribute name="VALUE" x="26.162" y="11.43" size="1.778" layer="96" rot="R90"/>
+</instance>
+<instance part="R7" gate="G$1" x="10.16" y="-25.4" smashed="yes">
+<attribute name="NAME" x="6.35" y="-23.9014" size="1.778" layer="95"/>
+<attribute name="VALUE" x="6.35" y="-28.702" size="1.778" layer="96"/>
+</instance>
+<instance part="Q1" gate="G$1" x="25.4" y="-25.4" smashed="yes">
+<attribute name="NAME" x="27.94" y="-25.4" size="1.778" layer="95" font="vector"/>
+<attribute name="VALUE" x="27.94" y="-27.686" size="1.778" layer="96" font="vector"/>
 </instance>
 </instances>
@@
 </segment>
 <segment>
-<pinref part="G" gate="G$1" pin="TP"/>
+<pinref part="IR-" gate="G$1" pin="TP"/>
 <wire x1="96.52" y1="-38.1" x2="96.52" y2="-33.02" width="0.1524" layer="91"/>
 <label x="96.52" y="-33.02" size="1.778" layer="95" rot="R90" xref="yes"/>
@@
 <label x="22.86" y="7.62" size="1.778" layer="95" xref="yes"/>
 </segment>
+<segment>
+<wire x1="27.94" y1="-30.48" x2="27.94" y2="-43.18" width="0.1524" layer="91"/>
+<label x="27.94" y="-43.18" size="1.778" layer="95"/>
+<pinref part="Q1" gate="G$1" pin="E"/>
+</segment>
+<segment>
+<pinref part="U1" gate="A" pin="3A"/>
+<wire x1="157.48" y1="53.34" x2="129.54" y2="53.34" width="0.1524" layer="91"/>
+<pinref part="U1" gate="A" pin="4A"/>
+<wire x1="157.48" y1="50.8" x2="129.54" y2="50.8" width="0.1524" layer="91"/>
+<wire x1="129.54" y1="50.8" x2="129.54" y2="53.34" width="0.1524" layer="91"/>
+<wire x1="129.54" y1="53.34" x2="124.46" y2="53.34" width="0.1524" layer="91"/>
+<junction x="129.54" y="53.34"/>
+<wire x1="124.46" y1="53.34" x2="124.46" y2="40.64" width="0.1524" layer="91"/>
+<label x="124.46" y="40.64" size="1.778" layer="95"/>
+</segment>
 </net>
 <net name="5V" class="2">
@@
 </segment>
 <segment>
-<pinref part="5V" gate="G$1" pin="TP"/>
+<pinref part="BZ+" gate="G$1" pin="TP"/>
 <wire x1="88.9" y1="-38.1" x2="88.9" y2="-33.02" width="0.1524" layer="91"/>
 <label x="88.9" y="-33.02" size="1.778" layer="95" rot="R90" xref="yes"/>
-</segment>
-<segment>
-<pinref part="R2" gate="G$1" pin="2"/>
-<wire x1="22.86" y1="30.48" x2="22.86" y2="33.02" width="0.1524" layer="91"/>
-<label x="22.86" y="33.02" size="1.778" layer="95"/>
 </segment>
 </net>
@@
 <net name="S1" class="0">
 <segment>
-<pinref part="BZ" gate="G$1" pin="TP"/>
-<wire x1="78.74" y1="-38.1" x2="78.74" y2="-30.48" width="0.1524" layer="91"/>
-<label x="78.74" y="-30.48" size="1.778" layer="95" rot="R90" xref="yes"/>
-</segment>
-<segment>
 <pinref part="B1" gate="G$1" pin="*5"/>
 <wire x1="55.88" y1="22.86" x2="48.26" y2="22.86" width="0.1524" layer="91"/>
 <label x="48.26" y="22.86" size="1.778" layer="95" rot="R180" xref="yes"/>
 </segment>
+<segment>
+<pinref part="R7" gate="G$1" pin="1"/>
+<wire x1="5.08" y1="-25.4" x2="-2.54" y2="-25.4" width="0.1524" layer="91"/>
+<label x="-2.54" y="-25.4" size="1.778" layer="95"/>
+</segment>
+</net>
+<net name="N$1" class="0">
+<segment>
+<pinref part="B1" gate="G$1" pin="*6"/>
+<pinref part="R2" gate="G$1" pin="2"/>
+<wire x1="55.88" y1="20.32" x2="35.56" y2="20.32" width="0.1524" layer="91"/>
+</segment>
 </net>
 <net name="3V" class="0">
@@
 <segment>
 <pinref part="R2" gate="G$1" pin="1"/>
+<wire x1="25.4" y1="20.32" x2="22.86" y2="20.32" width="0.1524" layer="91"/>
 <label x="17.78" y="20.32" size="1.778" layer="95" rot="R180" xref="yes"/>
 <pinref part="R6" gate="G$1" pin="2"/>
 <wire x1="22.86" y1="20.32" x2="17.78" y2="20.32" width="0.1524" layer="91"/>
 <junction x="22.86" y="20.32"/>
-<pinref part="B1" gate="G$1" pin="*6"/>
-<wire x1="22.86" y1="20.32" x2="55.88" y2="20.32" width="0.1524" layer="91"/>
 </segment>
 <segment>
@@
 </segment>
 </net>
+<net name="N$5" class="0">
+<segment>
+<pinref part="R7" gate="G$1" pin="2"/>
+<wire x1="15.24" y1="-25.4" x2="22.86" y2="-25.4" width="0.1524" layer="91"/>
+<pinref part="Q1" gate="G$1" pin="B"/>
+</segment>
+</net>
+<net name="BZ-" class="0">
+<segment>
+<wire x1="27.94" y1="-20.32" x2="27.94" y2="-15.24" width="0.1524" layer="91"/>
+<label x="27.94" y="-15.24" size="1.778" layer="95"/>
+<pinref part="Q1" gate="G$1" pin="C"/>
+</segment>
+<segment>
+<pinref part="BZ-" gate="G$1" pin="TP"/>
+<wire x1="78.74" y1="-38.1" x2="78.74" y2="-30.48" width="0.1524" layer="91"/>
+<label x="78.74" y="-30.48" size="1.778" layer="95" rot="R90" xref="yes"/>
+</segment>
+</net>

Commit message: Corrected PCB bug (IR diode)
Connections:
- removed net N$1: B1.*6, R2.2
- net 5V: now also R2.2
- net GND: now also IR+.TP; no longer IR-.TP
- net IR: now also B1.*6, IR-.TP; no longer IR+.TP
Other:
- moved on the sheet: IR+, IR-, R2, R6
Changed lines of the file:
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@@
 <part name="GND7" library="SparkFun-PowerSymbols" library_urn="urn:adsk.eagle:library:530" deviceset="GND" device=""/>
 <part name="C3" library="rcl" library_urn="urn:adsk.eagle:library:334" deviceset="C-EU" device="C1206" package3d_urn="urn:adsk.eagle:package:23618/2" value="100nf"/>
-<part name="IR+" library="testpad" library_urn="urn:adsk.eagle:library:385" deviceset="TP" device="TP15R" package3d_urn="urn:adsk.eagle:package:27968/1"/>
+<part name="IR-" library="testpad" library_urn="urn:adsk.eagle:library:385" deviceset="TP" device="TP15R" package3d_urn="urn:adsk.eagle:package:27968/1"/>
 <part name="U1" library="SN74HC4066D" deviceset="SN74HC4066D" device=""/>
 <part name="B1" library="SparkFun-Boards" deviceset="SPARKFUN_PRO_MICRO" device=""/>
@@
 <part name="BZ-" library="testpad" library_urn="urn:adsk.eagle:library:385" deviceset="TP" device="TP15R" package3d_urn="urn:adsk.eagle:package:27968/1"/>
 <part name="BZ+" library="testpad" library_urn="urn:adsk.eagle:library:385" deviceset="TP" device="TP15R" package3d_urn="urn:adsk.eagle:package:27968/1"/>
-<part name="IR-" library="testpad" library_urn="urn:adsk.eagle:library:385" deviceset="TP" device="TP15R" package3d_urn="urn:adsk.eagle:package:27968/1"/>
+<part name="IR+" library="testpad" library_urn="urn:adsk.eagle:library:385" deviceset="TP" device="TP15R" package3d_urn="urn:adsk.eagle:package:27968/1"/>
 <part name="R2" library="rcl" library_urn="urn:adsk.eagle:library:334" deviceset="R-EU_" device="R0603" package3d_urn="urn:adsk.eagle:package:23555/3" value="10k"/>
 <part name="R6" library="rcl" library_urn="urn:adsk.eagle:library:334" deviceset="R-EU_" device="R0603" package3d_urn="urn:adsk.eagle:package:23555/3" value="10k"/>
@@
 <attribute name="VALUE" x="263.779" y="-34.036" size="1.778" layer="96" rot="R90"/>
 </instance>
-<instance part="IR+" gate="G$1" x="71.12" y="-40.64" smashed="yes" rot="R180">
+<instance part="IR-" gate="G$1" x="71.12" y="-40.64" smashed="yes" rot="R180">
 <attribute name="NAME" x="72.39" y="-41.91" size="1.778" layer="95" rot="R180"/>
 <attribute name="TP_SIGNAL_NAME" x="69.85" y="-39.37" size="1.778" layer="97" rot="R180"/>
@@
 <attribute name="TP_SIGNAL_NAME" x="87.63" y="-39.37" size="1.778" layer="97" rot="R180"/>
 </instance>
-<instance part="IR-" gate="G$1" x="96.52" y="-40.64" smashed="yes" rot="R180">
+<instance part="IR+" gate="G$1" x="96.52" y="-40.64" smashed="yes" rot="R180">
 <attribute name="NAME" x="97.79" y="-41.91" size="1.778" layer="95" rot="R180"/>
 <attribute name="TP_SIGNAL_NAME" x="95.25" y="-39.37" size="1.778" layer="97" rot="R180"/>
 </instance>
-<instance part="R2" gate="G$1" x="30.48" y="20.32" smashed="yes">
-<attribute name="NAME" x="26.67" y="21.8186" size="1.778" layer="95"/>
-<attribute name="VALUE" x="26.67" y="17.018" size="1.778" layer="96"/>
-</instance>
-<instance part="R6" gate="G$1" x="22.86" y="15.24" smashed="yes" rot="R90">
-<attribute name="NAME" x="21.3614" y="11.43" size="1.778" layer="95" rot="R90"/>
-<attribute name="VALUE" x="26.162" y="11.43" size="1.778" layer="96" rot="R90"/>
+<instance part="R2" gate="G$1" x="10.16" y="5.08" smashed="yes">
+<attribute name="NAME" x="6.35" y="6.5786" size="1.778" layer="95"/>
+<attribute name="VALUE" x="6.35" y="1.778" size="1.778" layer="96"/>
+</instance>
+<instance part="R6" gate="G$1" x="2.54" y="0" smashed="yes" rot="R90">
+<attribute name="NAME" x="1.0414" y="-3.81" size="1.778" layer="95" rot="R90"/>
+<attribute name="VALUE" x="5.842" y="-3.81" size="1.778" layer="96" rot="R90"/>
 </instance>
 <instance part="R7" gate="G$1" x="10.16" y="-25.4" smashed="yes">
@@
 </segment>
 <segment>
-<pinref part="IR-" gate="G$1" pin="TP"/>
+<pinref part="IR+" gate="G$1" pin="TP"/>
 <wire x1="96.52" y1="-38.1" x2="96.52" y2="-33.02" width="0.1524" layer="91"/>
 <label x="96.52" y="-33.02" size="1.778" layer="95" rot="R90" xref="yes"/>
@@
 <segment>
 <pinref part="R6" gate="G$1" pin="1"/>
-<wire x1="22.86" y1="10.16" x2="22.86" y2="7.62" width="0.1524" layer="91"/>
-<label x="22.86" y="7.62" size="1.778" layer="95" xref="yes"/>
+<wire x1="2.54" y1="-5.08" x2="2.54" y2="-7.62" width="0.1524" layer="91"/>
+<label x="2.54" y="-7.62" size="1.778" layer="95" xref="yes"/>
 </segment>
 <segment>
@@
 <wire x1="88.9" y1="-38.1" x2="88.9" y2="-33.02" width="0.1524" layer="91"/>
 <label x="88.9" y="-33.02" size="1.778" layer="95" rot="R90" xref="yes"/>
+</segment>
+<segment>
+<pinref part="R2" gate="G$1" pin="2"/>
+<wire x1="15.24" y1="5.08" x2="20.32" y2="5.08" width="0.1524" layer="91"/>
+<label x="20.32" y="5.08" size="1.778" layer="95"/>
 </segment>
 </net>
@@
 </segment>
 </net>
-<net name="N$1" class="0">
-<segment>
-<pinref part="B1" gate="G$1" pin="*6"/>
-<pinref part="R2" gate="G$1" pin="2"/>
-<wire x1="55.88" y1="20.32" x2="35.56" y2="20.32" width="0.1524" layer="91"/>
-</segment>
-</net>
 <net name="3V" class="0">
 <segment>
@@
 <segment>
 <pinref part="R2" gate="G$1" pin="1"/>
-<wire x1="25.4" y1="20.32" x2="22.86" y2="20.32" width="0.1524" layer="91"/>
-<label x="17.78" y="20.32" size="1.778" layer="95" rot="R180" xref="yes"/>
+<wire x1="5.08" y1="5.08" x2="2.54" y2="5.08" width="0.1524" layer="91"/>
+<label x="-2.54" y="5.08" size="1.778" layer="95" rot="R180" xref="yes"/>
 <pinref part="R6" gate="G$1" pin="2"/>
-<wire x1="22.86" y1="20.32" x2="17.78" y2="20.32" width="0.1524" layer="91"/>
-<junction x="22.86" y="20.32"/>
-</segment>
-<segment>
-<pinref part="IR+" gate="G$1" pin="TP"/>
+<wire x1="2.54" y1="5.08" x2="-2.54" y2="5.08" width="0.1524" layer="91"/>
+<junction x="2.54" y="5.08"/>
+</segment>
+<segment>
+<pinref part="IR-" gate="G$1" pin="TP"/>
 <wire x1="71.12" y1="-38.1" x2="71.12" y2="-30.48" width="0.1524" layer="91"/>
 <label x="71.12" y="-30.48" size="1.778" layer="95" rot="R90" xref="yes"/>
 </segment>
-</net>
+<segment>
+<pinref part="B1" gate="G$1" pin="*6"/>
+<wire x1="55.88" y1="20.32" x2="48.26" y2="20.32" width="0.1524" layer="91"/>
+<label x="48.26" y="20.32" size="1.778" layer="95"/>
+</segment>
+</net>
